Commit message: Incomplete ros2_control

File: description/robot_core.xacro (robot description, xacro)
@@ -41,4 +41,7 @@
         </xacro:inertial_box>
     </link>
+    <gazebo reference = "left_wheel">
+        <material> Gazebo/White </material>
+    </gazebo>
     <!-- LEFT WHEEL LINK -->
     <joint name = "left_wheel_joint" type = "continuous">
@@ -64,4 +67,7 @@
         </xacro:inertial_cylinder>
     </link>
+    <gazebo reference = "left_wheel">
+        <material> Gazebo/Blue </material>
+    </gazebo>
     <!-- RIGHT WHEEL LINK -->
     <joint name = "right_wheel_joint" type = "continuous">
@@ -87,4 +93,7 @@
         </xacro:inertial_cylinder>
     </link>
+    <gazebo reference = "right_wheel">
+        <material> Gazebo/Blue </material>
+    </gazebo>
     <!--CASTOR WHEEL link-->
     <joint name = "castor_wheel_joint" type = "fixed">
@@ -109,3 +118,6 @@
         </xacro:inertial_sphere>
     </link>
+    <gazebo reference = "castor_wheel">
+        <material> Gazebo/Black </material>
+    </gazebo>
 </robot>
